File: drone-FC-v0.3/MCU.kicad_sch (KiCad schematic)
At the start: 11 parts, among them J11 USB_C_Receptacle_USB2.0_16P, U2 ESP32-S3-WROOM-1

Commit message: "Added Global Labels + deleted unnecessary parts on the PCB"
Connections:
- net GPIO 19 is gone; now on net USB_D-: D7.2 (A2), J11.A7 (D-), J11.B7 (D-)
- net GPIO 20 is gone; now on net USB_D+: D9.2 (A2), J11.A6 (D+), J11.B6 (D+)
Changed lines of the file:
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@@
+		)
+	)
+	(label "USB_D-"
+		(at 111.76 40.64 0)
+		(effects
+			(font
+				(size 1.27 1.27)
+			)
+			(justify left bottom)
 		)
 	)
@@
 	(label "UART_1_RX"
 		(at 243.84 50.8 0)
+		(effects
+			(font
+				(size 1.27 1.27)
+			)
+			(justify left bottom)
+		)
+	)
+	(label "USB_D+"
+		(at 111.76 45.72 0)
 		(effects
 			(font
@@
 		(effects
 			(font
-				(size 1.27 1.27)
-			)
-			(justify left bottom)
-		)
-	)
-	(label "GPIO 20"
-		(at 102.87 45.72 0)
-		(effects
-			(font
-				(size 1.27 1.27)
-			)
-			(justify left bottom)
-		)
-	)
-	(label "GPIO 19"
-		(at 102.87 40.64 0)
-		(effects
-			(font
